File: p2.sch (KiCad schematic (older format))
At the start: 26 parts, among them J1 BARREL_JACK, J2 FLASH_JMP, J3 UART, J4 ALT_Pwr, J5 jack-3.5mm-5pin, J6 jack-3.5mm-5pin, J7 jack-3.5mm-5pin, J8 jack-3.5mm-5pin, Q1 IRL540N, Q2 IRL540N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

Commit message: Backup old state
Parts:
- C2: symbol CP -> p2-rescue:CP
- C3, C4: symbol C -> p2-rescue:C
- D1, D2: symbol D -> p2-rescue:D
- J1: symbol BARREL_JACK -> p2-rescue:BARREL_JACK
- J2: symbol CONN_01X03 -> p2-rescue:CONN_01X03
- J3: symbol CONN_01X04 -> p2-rescue:CONN_01X04
- J4: symbol CONN_01X02 -> p2-rescue:CONN_01X02
- J5, J6, J7, J8: symbol jack-3.5mm-5pin -> p2-rescue:jack-3.5mm-5pin
- LED1, LED2: symbol LED -> p2-rescue:LED
- Q1, Q2: symbol IRL540N -> p2-rescue:IRL540N
- R3, R4, R5, R8, R9: symbol R -> p2-rescue:R
- RN1: symbol R_Network04 -> p2-rescue:R_Network04
- U1: symbol R-78E3.3-0.5 -> p2-rescue:R-78E3.3-0.5
- U2: symbol ESP-12 -> p2-rescue:ESP-12
- U3: symbol Switch -> p2-rescue:Switch
Changed lines of the file:
@@
-EESchema Schematic File Version 2
-LIBS:power
-LIBS:device
-LIBS:transistors
-LIBS:conn
-LIBS:linear
-LIBS:regul
-LIBS:74xx
-LIBS:cmos4000
-LIBS:adc-dac
-LIBS:memory
-LIBS:xilinx
-LIBS:microcontrollers
-LIBS:dsp
-LIBS:microchip
-LIBS:analog_switches
-LIBS:motorola
-LIBS:texas
-LIBS:intel
-LIBS:audio
-LIBS:interface
-LIBS:digital-audio
-LIBS:philips
-LIBS:display
-LIBS:cypress
-LIBS:siliconi
-LIBS:opto
-LIBS:atmel
-LIBS:contrib
-LIBS:valves
-LIBS:ESP8266
-LIBS:myschematics
+EESchema Schematic File Version 4
 LIBS:p2-cache
-EELAYER 25 0
+EELAYER 26 0
 EELAYER END
 $Descr A4 11693 8268
@@
 $EndDescr
 $Comp
-L BARREL_JACK J1
+L p2-rescue:BARREL_JACK J1
 U 1 1 58F61418
 P 1000 6950
@@
 $EndComp
 $Comp
-L D D2
+L p2-rescue:D D2
 U 1 1 58F61848
 P 9150 4950
@@
 $EndComp
 $Comp
-L D D1
+L p2-rescue:D D1
 U 1 1 58F619E5
 P 9150 4200
@@
 $EndComp
 $Comp
-L jack-3.5mm-5pin J5
+L p2-rescue:jack-3.5mm-5pin J5
 U 1 1 58FCB74A
 P 9450 1200
@@
 $EndComp
 $Comp
-L jack-3.5mm-5pin J6
+L p2-rescue:jack-3.5mm-5pin J6
 U 1 1 58FCC088
 P 9450 1900
@@
 $EndComp
 $Comp
-L jack-3.5mm-5pin J7
+L p2-rescue:jack-3.5mm-5pin J7
 U 1 1 58FCC0ED
 P 9800 4250
@@
 $EndComp
 $Comp
-L jack-3.5mm-5pin J8
+L p2-rescue:jack-3.5mm-5pin J8
 U 1 1 58FCC124
 P 9800 5000
@@
 ctl4
 $Comp
-L GNDREF #PWR01
+L p2-rescue:GNDREF #PWR01
 U 1 1 58FCE5D7
 P 8600 6000
@@
 $EndComp
 $Comp
-L R R4
+L p2-rescue:R R4
 U 1 1 58FCE6F3
 P 8150 4600
@@
 $EndComp
 $Comp
-L R R5
+L p2-rescue:R R5
 U 1 1 58FCE75E
 P 8150 5350
@@
 NoConn ~ 9200 1100
 $Comp
-L GNDREF #PWR02
+L p2-rescue:GNDREF #PWR02
 U 1 1 58FCF0DE
 P 9050 2650
@@
 ctl2
 $Comp
-L R R3
+L p2-rescue:R R3
 U 1 1 58FCF9B3
 P 6150 7450
@@
 $EndComp
 $Comp
-L GNDREF #PWR03
+L p2-rescue:GNDREF #PWR03
 U 1 1 58FCFA4D
 P 5700 2850
@@
 $EndComp
 $Comp
-L C C4
+L p2-rescue:C C4
 U 1 1 58FCFEB0
 P 4550 1400
@@
 Vcc
 $Comp
-L GNDREF #PWR04
+L p2-rescue:GNDREF #PWR04
 U 1 1 58FCFF82
 P 3650 1250
@@
 GND
 $Comp
-L GNDREF #PWR05
+L p2-rescue:GNDREF #PWR05
 U 1 1 58FD2360
 P 2850 7150
@@
 $EndComp
 $Comp
-L CP C2
+L p2-rescue:CP C2
 U 1 1 58FD1361
 P 2500 7000
@@
 $EndComp
 $Comp
-L C C3
+L p2-rescue:C C3
 U 1 1 58FD1608
 P 4150 1400
@@
 GND
 $Comp
-L CONN_01X02 J4
+L p2-rescue:CONN_01X02 J4
 U 1 1 58FD0660
 P 1200 5050
@@
 $EndComp
 $Comp
-L CONN_01X03 J2
+L p2-rescue:CONN_01X03 J2
 U 1 1 58FD04F7
 P 1200 1300
@@
 $EndComp
 $Comp
-L CONN_01X04 J3
+L p2-rescue:CONN_01X04 J3
 U 1 1 58FD0298
 P 1200 3250
@@
 NoConn ~ 9550 5200
 $Comp
-L IRL540N Q1
+L p2-rescue:IRL540N Q1
 U 1 1 58FD3732
 P 8500 4550
@@
 $EndComp
 $Comp
-L IRL540N Q2
+L p2-rescue:IRL540N Q2
 U 1 1 58FD3779
 P 8500 5300
@@
 Pump Controls
 $Comp
-L LED LED2
+L p2-rescue:LED LED2
 U 1 1 5904F834
 P 4300 7500
@@
 $EndComp
 $Comp
-L LED LED1
+L p2-rescue:LED LED1
 U 1 1 5904FA17
 P 4300 7150
@@
 $EndComp
 $Comp
-L GNDREF #PWR06
+L p2-rescue:GNDREF #PWR06
 U 1 1 5904FBC6
 P 4800 7350
@@
 $EndComp
 $Comp
-L R R8
+L p2-rescue:R R8
 U 1 1 5904FDAC
 P 4000 7500
@@
 $EndComp
 $Comp
-L R R9
+L p2-rescue:R R9
 U 1 1 5904FE63
 P 4000 7150
@@
 $EndComp
 $Comp
-L +3.3V #PWR07
+L p2-rescue:+3.3V #PWR07
 U 1 1 59050FF8
 P 6150 6700
@@
 $EndComp
 $Comp
-L +3.3V #PWR08
+L p2-rescue:+3.3V #PWR08
 U 1 1 59051972
 P 2650 6850
@@
 $EndComp
 $Comp
-L +3.3V #PWR09
+L p2-rescue:+3.3V #PWR09
 U 1 1 590519E1
 P 2650 6850
@@
 2 signal LEDs
 Wire Wire Line
-	9150 4800 9550 4800
-Wire Wire Line
-	9150 4050 9550 4050
-Wire Wire Line
-	1300 6850 1700 6850
+	9150 4800 9300 4800
+Wire Wire Line
+	9150 4050 9300 4050
+Wire Wire Line
+	1300 6850 1550 6850
 Wire Wire Line
 	1300 7050 1300 7150
@@
 	1550 6850 1550 6500
 Wire Wire Line
-	1550 6500 2850 6500
+	1550 6500 2650 6500
 Connection ~ 1550 6850
 Wire Wire Line
-	2300 6850 2850 6850
+	2300 6850 2500 6850
 Connection ~ 2500 6850
 Connection ~ 2500 7150
@@
 	8450 1300 9200 1300
 Wire Wire Line
-	9050 1000 9050 2650
+	9050 1000 9050 1700
 Wire Wire Line
 	9050 1700 9200 1700
@@
 Connection ~ 9150 4350
 Wire Wire Line
-	9300 4050 9300 6100
+	9300 4050 9300 4800
 Connection ~ 9300 4800
 Connection ~ 9300 4050
 Wire Wire Line
-	3400 1650 4150 1650
+	3400 1650 3950 1650
 Connection ~ 4550 1650
 Wire Wire Line
-	3650 1250 4550 1250
+	3650 1250 4150 1250
 Wire Wire Line
 	3700 2150 4800 2150
@@
 Wire Wire Line
 	1900 5000 1400 5000
-Connection ~ 8600 6000
-Connection ~ 2850 7150
-Wire Wire Line
-	8600 4350 9550 4350
-Wire Wire Line
-	8600 5100 9550 5100
-Wire Notes Line
-	3150 500  3150 7800
+Wire Wire Line
+	8600 4350 9150 4350
+Wire Wire Line
+	8600 5100 9150 5100
 Wire Notes Line
 	500  6000 3150 6000
-Wire Notes Line
-	3150 6000 3150 6050
 Wire Notes Line
 	500  4300 3150 4300
@@
 	4450 7500 4600 7500
 Wire Wire Line
-	4600 7500 4600 7150
+	4600 7500 4600 7350
 Wire Wire Line
 	4600 7150 4450 7150
@@
 	3150 6500 7250 6500
 $Comp
-L Switch U3
+L p2-rescue:Switch U3
 U 1 1 59051246
 P 6300 7000
@@
 led1
 $Comp
-L ESP-12 U2
+L p2-rescue:ESP-12 U2
 U 1 1 590CA322
 P 5700 1950
@@
 pump2
 $Comp
-L R-78E3.3-0.5 U1
+L p2-rescue:R-78E3.3-0.5 U1
 U 1 1 59126417
 P 2000 6850
@@
 Connection ~ 6150 7300
 $Comp
-L GNDREF #PWR010
+L p2-rescue:GNDREF #PWR010
 U 1 1 59127D38
 P 6150 7600
@@
 wifi-switch
 Wire Wire Line
-	1300 7150 2850 7150
+	1300 7150 2000 7150
 NoConn ~ 4800 1750
 $Comp
-L R_Network04 RN1
+L p2-rescue:R_Network04 RN1
 U 1 1 5922FA0C
 P 4350 1750
@@
 	4800 1950 4700 1950
 Wire Wire Line
-	4700 1850 4700 2600
+	4700 1850 4700 1950
 Wire Wire Line
 	4700 1850 4550 1850
@@
 	4600 2050 4800 2050
 Wire Wire Line
-	4600 1950 4600 2600
+	4600 1950 4600 2050
 Wire Wire Line
 	4600 1950 4550 1950
@@
 Connection ~ 4600 2050
 Wire Wire Line
-	4150 1550 4150 1950
-$Comp
-L +12V #PWR011
+	4150 1550 4150 1650
+$Comp
+L p2-rescue:+12V #PWR011
 U 1 1 5923129E
 P 2650 6500
@@
 $EndComp
 Connection ~ 2650 6500
+Wire Wire Line
+	1550 6850 1700 6850
+Wire Wire Line
+	2500 6850 2650 6850
+Wire Wire Line
+	2500 7150 2850 7150
+Wire Wire Line
+	9050 1700 9050 2650
+Wire Wire Line
+	9150 5100 9550 5100
+Wire Wire Line
+	9150 4350 9550 4350
+Wire Wire Line
+	9300 4800 9550 4800
+Wire Wire Line
+	9300 4800 9300 6100
+Wire Wire Line
+	9300 4050 9550 4050
+Wire Wire Line
+	4150 1650 4150 1950
+Wire Wire Line
+	4150 1250 4550 1250
+Wire Wire Line
+	2000 7150 2500 7150
+Wire Wire Line
+	4600 7350 4600 7150
+Wire Wire Line
+	2650 6850 2850 6850
+Wire Wire Line
+	3950 1650 4150 1650
+Wire Wire Line
+	4700 1950 4700 2600
+Wire Wire Line
+	4600 2050 4600 2600
+Wire Wire Line
+	2650 6500 2850 6500
+Wire Notes Line
+	3150 500  3150 7800
 $EndSCHEMATC
